Commit message: Initial commnit

File: install/rmitbot_description/share/rmitbot_description/urdf/rmitbot_ros2_control.xacro (robot description, xacro)
@@ -16,5 +16,5 @@
         </xacro:unless>
         <!-- ros2_control Common Interfaces -->
-        <joint name="wheel_right_joint">
+        <joint name="front_right_wheel_joint">
             <command_interface name="velocity">
                 <param name="min">-1</param>
@@ -24,5 +24,21 @@
             <state_interface name="velocity" />
         </joint>
-        <joint name="wheel_left_joint">
+        <joint name="front_left_wheel_joint">
+            <command_interface name="velocity">
+                <param name="min">-1</param>
+                <param name="max">1</param>
+            </command_interface>
+            <state_interface name="position" />
+            <state_interface name="velocity" />
+        </joint>
+        <joint name="rear_right_wheel_joint">
+            <command_interface name="velocity">
+                <param name="min">-1</param>
+                <param name="max">1</param>
+            </command_interface>
+            <state_interface name="position" />
+            <state_interface name="velocity" />
+        </joint>
+        <joint name="rear_left_wheel_joint">
             <command_interface name="velocity">
                 <param name="min">-1</param>
@@ -33,3 +49,9 @@
         </joint>
     </ros2_control>
+    <!-- ROS 2 Control Gazebo plugins -->
+    <gazebo>
+        <plugin filename="gz_ros2_control-system" name="gz_ros2_control::GazeboSimROS2ControlPlugin">
+            <parameters>$(find rmitbot_controller)/config/rmitbot_controller.yaml</parameters>
+        </plugin>
+    </gazebo>
 </robot>

File: src/rmitbot_description/urdf/rmitbot_ros2_control.xacro (robot description, xacro)
@@ -16,5 +16,5 @@
         </xacro:unless>
         <!-- ros2_control Common Interfaces -->
-        <joint name="wheel_right_joint">
+        <joint name="front_right_wheel_joint">
             <command_interface name="velocity">
                 <param name="min">-1</param>
@@ -24,5 +24,21 @@
             <state_interface name="velocity" />
         </joint>
-        <joint name="wheel_left_joint">
+        <joint name="front_left_wheel_joint">
+            <command_interface name="velocity">
+                <param name="min">-1</param>
+                <param name="max">1</param>
+            </command_interface>
+            <state_interface name="position" />
+            <state_interface name="velocity" />
+        </joint>
+        <joint name="rear_right_wheel_joint">
+            <command_interface name="velocity">
+                <param name="min">-1</param>
+                <param name="max">1</param>
+            </command_interface>
+            <state_interface name="position" />
+            <state_interface name="velocity" />
+        </joint>
+        <joint name="rear_left_wheel_joint">
             <command_interface name="velocity">
                 <param name="min">-1</param>
